File: kbd60.kicad_sch (KiCad schematic)
At the start: 164 parts, among them J1 5077CR-16-SMC2-BK-TR, SW1 ESC, SW10 9, SW11 0, SW12 -, SW13 =, SW14 Backspace, SW15 Tab, SW16 Q, SW17 W, SW18 E, SW19 R, SW2 1, SW20 T, SW21 Y, SW22 U, SW23 I, SW24 O, SW25 P, SW26 [, SW27 ], SW28 \, SW29 CapsLock, SW3 2, SW30 A, SW31 S, SW32 D, SW33 F, SW34 G, SW35 H, SW36 J, SW37 K, SW38 L, SW39 ;, SW4 3, SW40 ', SW41 Enter, SW42 ShiftL, SW43 Z, SW44 X, SW45 C, SW46 V, SW47 B, SW48 N, SW49 M, SW5 4, SW50 ,, SW51 ., SW52 /, SW53 ShiftR, SW54 CtrlL, SW55 SuperL, SW56 AltL, SW57 Space, SW58 Fn, SW59 SuperR, SW6 5, SW60 AltR, SW61 CtrlR, SW7 6, SW8 7, SW9 8, U1 RP2040, U2 NJM12877F33, U3 W25Q16JVUXIQ, Y1 FA238V

Commit message: wip: update F.Cu
Connections:
- net SHIELD: now reaches C18.1, J1.S1 (SHIELD), R12.1
Changed lines of the file:
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@@
+    (effects (font (size 1.27 1.27)) (justify right bottom))
+  )
+  (label "SHIELD" (at 39.37 242.57 180) (fields_autoplaced)
     (effects (font (size 1.27 1.27)) (justify right bottom))
   )

Commit message: wip: update footprint libs
Parts:
- SW1, SW10, SW11, SW12, SW13, SW16, SW17, SW18, SW19, SW2, SW20, SW21, SW22, SW23, SW24, SW25, SW26, SW27, SW3, SW30, SW31, SW32, SW33, SW34, SW35, SW36, SW37, SW38, SW39, SW4, SW40, SW43, SW44, SW45, SW46, SW47, SW48, SW49, SW5, SW50, SW51, SW52, SW6, SW7, SW8, SW9: footprint PCM_Switch_Keyboard_Cherry_MX:SW_Cherry_MX_PCB_1.00u -> Button_Switch_Keyboard:SW_Cherry_MX_1.00u_PCB
- SW14: footprint PCM_Switch_Keyboard_Cherry_MX:SW_Cherry_MX_PCB_2.00u -> Button_Switch_Keyboard:SW_Cherry_MX_2.00u_PCB
- SW15, SW28: footprint PCM_Switch_Keyboard_Cherry_MX:SW_Cherry_MX_PCB_1.50u -> Button_Switch_Keyboard:SW_Cherry_MX_1.50u_PCB
- SW29: footprint PCM_Switch_Keyboard_Cherry_MX:SW_Cherry_MX_PCB_1.75u -> Button_Switch_Keyboard:SW_Cherry_MX_1.75u_PCB
- SW41, SW42: footprint PCM_Switch_Keyboard_Cherry_MX:SW_Cherry_MX_PCB_2.25u -> Button_Switch_Keyboard:SW_Cherry_MX_2.25u_PCB
- SW53: footprint PCM_Switch_Keyboard_Cherry_MX:SW_Cherry_MX_PCB_2.75u -> Button_Switch_Keyboard:SW_Cherry_MX_2.75u_PCB
- SW54, SW55, SW56, SW58, SW59, SW60, SW61: footprint PCM_Switch_Keyboard_Cherry_MX:SW_Cherry_MX_PCB_1.25u -> Button_Switch_Keyboard:SW_Cherry_MX_1.25u_PCB
- SW57: footprint PCM_Switch_Keyboard_Cherry_MX:SW_Cherry_MX_PCB_6.25u -> Button_Switch_Keyboard:SW_Cherry_MX_6.25u_PCB
Connections:
- net COL1: now also SW1.2, SW15.2, SW29.2, SW42.2, SW54.2; no longer SW1.1, SW15.1, SW29.1, SW42.1, SW54.1
- net COL10: now also SW10.2, SW24.2, SW38.2, SW51.2, SW58.2; no longer SW10.1, SW24.1, SW38.1, SW51.1, SW58.1
- net COL11: now also SW11.2, SW25.2, SW39.2, SW52.2, SW59.2; no longer SW11.1, SW25.1, SW39.1, SW52.1, SW59.1
- net COL12: now also SW12.2, SW26.2, SW40.2; no longer SW12.1, SW26.1, SW40.1
- net COL13: now also SW13.2, SW27.2, SW41.2, SW53.2, SW60.2; no longer SW13.1, SW27.1, SW41.1, SW53.1, SW60.1
- net COL14: now also SW14.2, SW28.2, SW61.2; no longer SW14.1, SW28.1, SW61.1
- net COL2: now also SW16.2, SW2.2, SW30.2, SW43.2, SW55.2; no longer SW16.1, SW2.1, SW30.1, SW43.1, SW55.1
- net COL3: now also SW17.2, SW3.2, SW31.2, SW44.2, SW56.2; no longer SW17.1, SW3.1, SW31.1, SW44.1, SW56.1
- net COL4: now also SW18.2, SW32.2, SW4.2, SW45.2; no longer SW18.1, SW32.1, SW4.1, SW45.1
- net COL5: now also SW19.2, SW33.2, SW46.2, SW5.2; no longer SW19.1, SW33.1, SW46.1, SW5.1
- net COL6: now also SW20.2, SW34.2, SW47.2, SW57.2, SW6.2; no longer SW20.1, SW34.1, SW47.1, SW57.1, SW6.1
- net COL7: now also SW21.2, SW35.2, SW48.2, SW7.2; no longer SW21.1, SW35.1, SW48.1, SW7.1
- net COL8: now also SW22.2, SW36.2, SW49.2, SW8.2; no longer SW22.1, SW36.1, SW49.1, SW8.1
- net COL9: now also SW23.2, SW37.2, SW50.2, SW9.2; no longer SW23.1, SW37.1, SW50.1, SW9.1
- net at D31.2 (A): now also SW31.1; no longer SW31.2
- net at D15.2 (A): now also SW15.1; no longer SW15.2
- net at D23.2 (A): now also SW23.1; no longer SW23.2
- net at D25.2 (A): now also SW25.1; no longer SW25.2
- net at D37.2 (A): now also SW37.1; no longer SW37.2
- net at D8.2 (A): now also SW8.1; no longer SW8.2
- net at D9.2 (A): now also SW9.1; no longer SW9.2
- net at D6.2 (A): now also SW6.1; no longer SW6.2
- net at D20.2 (A): now also SW20.1; no longer SW20.2
- net at D39.2 (A): now also SW39.1; no longer SW39.2
- net at D16.2 (A): now also SW16.1; no longer SW16.2
- net at D60.2 (A): now also SW60.1; no longer SW60.2
- net at D26.2 (A): now also SW26.1; no longer SW26.2
- net at D12.2 (A): now also SW12.1; no longer SW12.2
- net at D54.2 (A): now also SW54.1; no longer SW54.2
- net at D35.2 (A): now also SW35.1; no longer SW35.2
- net at D61.2 (A): now also SW61.1; no longer SW61.2
- net at D47.2 (A): now also SW47.1; no longer SW47.2
- net at D7.2 (A): now also SW7.1; no longer SW7.2
- net at D10.2 (A): now also SW10.1; no longer SW10.2
- net at D51.2 (A): now also SW51.1; no longer SW51.2
- net at D36.2 (A): now also SW36.1; no longer SW36.2
- net at D22.2 (A): now also SW22.1; no longer SW22.2
- net at D48.2 (A): now also SW48.1; no longer SW48.2
- net at D13.2 (A): now also SW13.1; no longer SW13.2
- net at D11.2 (A): now also SW11.1; no longer SW11.2
- net at D1.2 (A): now also SW1.1; no longer SW1.2
- net at D57.2 (A): now also SW57.1; no longer SW57.2
- net at D14.2 (A): now also SW14.1; no longer SW14.2
- net at D45.2 (A): now also SW45.1; no longer SW45.2
- net at D33.2 (A): now also SW33.1; no longer SW33.2
- net at D52.2 (A): now also SW52.1; no longer SW52.2
- net at D5.2 (A): now also SW5.1; no longer SW5.2
- net at D19.2 (A): now also SW19.1; no longer SW19.2
- net at D24.2 (A): now also SW24.1; no longer SW24.2
- net at D55.2 (A): now also SW55.1; no longer SW55.2
- net at D21.2 (A): now also SW21.1; no longer SW21.2
- net at D42.2 (A): now also SW42.1; no longer SW42.2
- net at D59.2 (A): now also SW59.1; no longer SW59.2
- net at D18.2 (A): now also SW18.1; no longer SW18.2
- net at D46.2 (A): now also SW46.1; no longer SW46.2
- net at D44.2 (A): now also SW44.1; no longer SW44.2
- net at D2.2 (A): now also SW2.1; no longer SW2.2
- net at D34.2 (A): now also SW34.1; no longer SW34.2
- net at D4.2 (A): now also SW4.1; no longer SW4.2
- net at D58.2 (A): now also SW58.1; no longer SW58.2
- net at D56.2 (A): now also SW56.1; no longer SW56.2
- net at D43.2 (A): now also SW43.1; no longer SW43.2
- net at D41.2 (A): now also SW41.1; no longer SW41.2
- net at D50.2 (A): now also SW50.1; no longer SW50.2
- net at D53.2 (A): now also SW53.1; no longer SW53.2
- net at D30.2 (A): now also SW30.1; no longer SW30.2
- net at D17.2 (A): now also SW17.1; no longer SW17.2
- net at D38.2 (A): now also SW38.1; no longer SW38.2
- net at D29.2 (A): now also SW29.1; no longer SW29.2
- net at D32.2 (A): now also SW32.1; no longer SW32.2
- net at D27.2 (A): now also SW27.1; no longer SW27.2
- net at D49.2 (A): now also SW49.1; no longer SW49.2
- net at D28.2 (A): now also SW28.1; no longer SW28.2
- net at D3.2 (A): now also SW3.1; no longer SW3.2
- net at D40.2 (A): now also SW40.1; no longer SW40.2

Commit message: add mount holes
Parts:
- added H1, H2, H3, H4, H5, H6: M2.5, MountingHole:MountingHole_2.7mm_M2.5_ISO7380, symbol Mechanical:MountingHole
Connections:
- no-connect marks 8 -> 11
Changed lines of the file:
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@@
   (junction (at 231.14 45.72) (diameter 0) (color 0 0 0 0)
   )
+  (no_connect (at 365.76 105.41))
   (no_connect (at 365.76 153.67))
   (no_connect (at 365.76 151.13))
   (no_connect (at 365.76 156.21))
+  (no_connect (at 365.76 107.95))
+  (no_connect (at 365.76 102.87))
   (no_connect (at 314.96 151.13))
   (no_connect (at 62.23 228.6))
@@
     )
   )
+  (symbol (lib_id "Mechanical:MountingHole") (at 330.2 241.3 0) (unit 1)
+    (in_bom yes) (on_board yes) (dnp no) (fields_autoplaced)
+    (property "Reference" "H1" (at 332.74 240.03 0)
+      (effects (font (size 1.27 1.27)) (justify left))
+    )
+    (property "Value" "M2.5" (at 332.74 242.57 0)
+      (effects (font (size 1.27 1.27)) (justify left))
+    )
+    (property "Footprint" "MountingHole:MountingHole_2.7mm_M2.5_ISO7380" (at 330.2 241.3 0)
+      (effects (font (size 1.27 1.27)) hide)
+    )
+    (property "Datasheet" "~" (at 330.2 241.3 0)
+      (effects (font (size 1.27 1.27)) hide)
+    )
+    (instances
+      (project "kbd60"
+        (path "/f215fcda-e86a-40b0-a9f7-5dc893df6659"
+          (reference "H1") (unit 1)
+        )
+      )
+    )
+  )
   (symbol (lib_id "Device:D") (at 260.35 151.13 270) (mirror x) (unit 1)
     (in_bom yes) (on_board yes) (dnp no)
@@
     )
   )
+  (symbol (lib_id "Mechanical:MountingHole") (at 393.7 241.3 0) (unit 1)
+    (in_bom yes) (on_board yes) (dnp no) (fields_autoplaced)
+    (property "Reference" "H6" (at 396.24 240.03 0)
+      (effects (font (size 1.27 1.27)) (justify left))
+    )
+    (property "Value" "M2.5" (at 396.24 242.57 0)
+      (effects (font (size 1.27 1.27)) (justify left))
+    )
+    (property "Footprint" "MountingHole:MountingHole_2.7mm_M2.5_ISO7380" (at 393.7 241.3 0)
+      (effects (font (size 1.27 1.27)) hide)
+    )
+    (property "Datasheet" "~" (at 393.7 241.3 0)
+      (effects (font (size 1.27 1.27)) hide)
+    )
+    (instances
+      (project "kbd60"
+        (path "/f215fcda-e86a-40b0-a9f7-5dc893df6659"
+          (reference "H6") (unit 1)
+        )
+      )
+    )
+  )
   (symbol (lib_id "Switch:SW_Push") (at 102.87 96.52 0) (mirror y) (unit 1)
     (in_bom yes) (on_board yes) (dnp no) (fields_autoplaced)
@@
     )
   )
+  (symbol (lib_id "Mechanical:MountingHole") (at 342.9 241.3 0) (unit 1)
+    (in_bom yes) (on_board yes) (dnp no) (fields_autoplaced)
+    (property "Reference" "H2" (at 345.44 240.03 0)
+      (effects (font (size 1.27 1.27)) (justify left))
+    )
+    (property "Value" "M2.5" (at 345.44 242.57 0)
+      (effects (font (size 1.27 1.27)) (justify left))
+    )
+    (property "Footprint" "MountingHole:MountingHole_2.7mm_M2.5_ISO7380" (at 342.9 241.3 0)
+      (effects (font (size 1.27 1.27)) hide)
+    )
+    (property "Datasheet" "~" (at 342.9 241.3 0)
+      (effects (font (size 1.27 1.27)) hide)
+    )
+    (instances
+      (project "kbd60"
+        (path "/f215fcda-e86a-40b0-a9f7-5dc893df6659"
+          (reference "H2") (unit 1)
+        )
+      )
+    )
+  )
   (symbol (lib_id "Device:D") (at 203.2 151.13 270) (mirror x) (unit 1)
     (in_bom yes) (on_board yes) (dnp no)
@@
     )
   )
+  (symbol (lib_id "Mechanical:MountingHole") (at 355.6 241.3 0) (unit 1)
+    (in_bom yes) (on_board yes) (dnp no) (fields_autoplaced)
+    (property "Reference" "H3" (at 358.14 240.03 0)
+      (effects (font (size 1.27 1.27)) (justify left))
+    )
+    (property "Value" "M2.5" (at 358.14 242.57 0)
+      (effects (font (size 1.27 1.27)) (justify left))
+    )
+    (property "Footprint" "MountingHole:MountingHole_2.7mm_M2.5_ISO7380" (at 355.6 241.3 0)
+      (effects (font (size 1.27 1.27)) hide)
+    )
+    (property "Datasheet" "~" (at 355.6 241.3 0)
+      (effects (font (size 1.27 1.27)) hide)
+    )
+    (instances
+      (project "kbd60"
+        (path "/f215fcda-e86a-40b0-a9f7-5dc893df6659"
+          (reference "H3") (unit 1)
+        )
+      )
+    )
+  )
   (symbol (lib_id "Device:D") (at 107.95 100.33 270) (mirror x) (unit 1)
     (in_bom yes) (on_board yes) (dnp no)
@@
     )
   )
+  (symbol (lib_id "Mechanical:MountingHole") (at 368.3 241.3 0) (unit 1)
+    (in_bom yes) (on_board yes) (dnp no) (fields_autoplaced)
+    (property "Reference" "H4" (at 370.84 240.03 0)
+      (effects (font (size 1.27 1.27)) (justify left))
+    )
+    (property "Value" "M2.5" (at 370.84 242.57 0)
+      (effects (font (size 1.27 1.27)) (justify left))
+    )
+    (property "Footprint" "MountingHole:MountingHole_2.7mm_M2.5_ISO7380" (at 368.3 241.3 0)
+      (effects (font (size 1.27 1.27)) hide)
+    )
+    (property "Datasheet" "~" (at 368.3 241.3 0)
+      (effects (font (size 1.27 1.27)) hide)
+    )
+    (instances
+      (project "kbd60"
+        (path "/f215fcda-e86a-40b0-a9f7-5dc893df6659"
+          (reference "H4") (unit 1)
+        )
+      )
+    )
+  )
   (symbol (lib_id "Device:D") (at 260.35 74.93 270) (mirror x) (unit 1)
     (in_bom yes) (on_board yes) (dnp no)
@@
         )
       )
+    )
+  )
+  (symbol (lib_id "Mechanical:MountingHole") (at 381 241.3 0) (unit 1)
+    (in_bom yes) (on_board yes) (dnp no) (fields_autoplaced)
+    (property "Reference" "H5" (at 383.54 240.03 0)
+      (effects (font (size 1.27 1.27)) (justify left))
+    )
+    (property "Value" "M2.5" (at 383.54 242.57 0)
+      (effects (font (size 1.27 1.27)) (justify left))
+    )
+    (property "Footprint" "MountingHole:MountingHole_2.7mm_M2.5_ISO7380" (at 381 241.3 0)
+      (effects (font (size 1.27 1.27)) hide)
+    )
+    (property "Datasheet" "~" (at 381 241.3 0)
+      (effects (font (size 1.27 1.27)) hide)
+    )
+    (instances
+      (project "kbd60"
+        (path "/f215fcda-e86a-40b0-a9f7-5dc893df6659"
+          (reference "H5") (unit 1)
+        )
+      )
